Commit message: :heavy_check_mark: add ros2-ackermann custom package

File: ros2-packages/ros2-ackermann/src/description/ackermann_description.urdf (robot description, URDF)
Before this commit: robot wheeltec_robot, 5 links, 4 joints
Links:
- added link base_footprint
- added link laser_link; visual cylinder length=0.02 radius=0.05
Joints:
- added joint base_joint: type fixed, parent base_link, child base_footprint, origin xyz=0 0 0 rpy=0 0 0, axis 0 1 0
- added joint laser_joint: type fixed, parent base_link, child laser_link, origin xyz=0.52 0.0 0.35 rpy=0 0 0, axis 0 0 0

Commit message: :heavy_check_mark: fix laser_link

File: ros2-packages/ros2-ackermann/src/description/ackermann_description.urdf (robot description, URDF)
Before this commit: robot wheeltec_ackermann, 7 links, 6 joints
Links:
- removed link base_footprint
- link laser_link: geometry visual cylinder length=0.02 radius=0.035
Joints:
- removed joint base_joint
- joint laser_joint: origin xyz=0.52 0.0 0.35 rpy=0 0 0 -> xyz=0.265 0.0 0.16 rpy=0 0 0
- joint left_front_joint: origin xyz=0.53 0.295 0.12 rpy=1.57 0 0 -> xyz=0.275 0.295 -0.07 rpy=1.57 0 0
- joint left_wheel_joint: origin xyz=-0 0.295 0.12 rpy=1.57 0 0 -> xyz=-0.255 0.295 -0.07 rpy=1.57 0 0
- joint right_front_joint: origin xyz=0.53 -0.295 0.12 rpy=1.57 0 0 -> xyz=0.275 -0.295 -0.07 rpy=1.57 0 0
- joint right_wheel_joint: origin xyz=-0 -0.295 0.12 rpy=1.57 0 0 -> xyz=-0.255 -0.295 -0.07 rpy=1.57 0 0

Commit message: :heavy_check_mark: add ros2-ackermann custom package

File: ros2-packages/ros2-ackermann/src/description/ackermann_description.urdf (robot description, URDF)
Before this commit: robot wheeltec_ackermann, 6 links, 5 joints
Links:
- removed link left_front_link
- removed link left_wheel_link
- removed link right_front_link
- removed link right_wheel_link
- added link base_footprint
- link base_link: geometry visual box size=${base_length} ${base_width} ${base_height}
Joints:
- removed joint left_front_joint
- removed joint left_wheel_joint
- removed joint right_front_joint
- removed joint right_wheel_joint
- added joint base_joint: type fixed, parent base_link, child base_footprint, origin xyz=0.0 0.0 ${-(wheel_radius+wheel_zoff)} rpy=0 0 0

Commit message: :hammer: fix ros2-ackermann custom package

File: ros2-packages/ros2-ackermann/src/description/ackermann_description.urdf (robot description, URDF)
Before this commit: robot wheeltec_ackermann, 3 links, 2 joints
Joints:
- joint laser_joint: origin xyz=0.265 0.0 0.16 rpy=0 0 0 -> xyz=-0.265 0.0 0.16 rpy=0 0 0

Commit message: :hammer: fix urdf

File: ros2-packages/ros2-ackermann/src/description/ackermann_description.urdf (robot description, URDF)
Before this commit: robot wheeltec_ackermann, 3 links, 2 joints
Joints:
- joint laser_joint: origin xyz=-0.265 0.0 0.16 rpy=0 0 0 -> xyz=0.265 0.0 0.16 rpy=0 0 0
