Commit message: :recycle: refactor unity robot frames

File: ros2-packages/rhcr-slam-nav2/src/description/unity_ackermann_description.urdf (robot description, URDF)
Before this commit: robot wheeltec_ackermann, 3 links, 2 joints
Links:
- removed link base_footprint
- removed link base_link
- removed link laser_link
- added link unity_base_footprint
- added link unity_base_link; visual box size=${base_length} ${base_width} ${base_height}
- added link unity_laser_link; visual cylinder length=0.02 radius=0.035
Joints:
- removed joint base_joint
- removed joint laser_joint
- added joint unity_base_joint: type fixed, parent unity_base_link, child unity_base_footprint, origin xyz=0.0 0.0 ${-(wheel_radius+wheel_zoff)} rpy=0 0 0
- added joint unity_laser_joint: type fixed, parent unity_base_link, child unity_laser_link, origin xyz=0.265 0.0 0.16 rpy=0 0 0, axis 0 0 0
